Commit message: added lidar to jackal-urdf

File: catkin_ws/src/jackal_realsense/jackal_realsense.urdf.xacro (robot description, xacro)
@@ -2,9 +2,4 @@
 <robot xmlns:xacro="http://ros.org/wiki/xacro">
   <link name="front_realsense" />
-  <!--
-    The gazebo plugin aligns the depth data with the Z axis, with X=left and Y=up
-    ROS expects the depth data along the X axis, with Y=left and Z=up
-    This link only exists to give the gazebo plugin the correctly-oriented frame
-  -->
   <link name="front_realsense_gazebo" />
   <joint name="front_realsense_gazebo_joint" type="fixed">
@@ -18,5 +13,4 @@
       <update_rate>30</update_rate>
       <camera>
-        <!-- 75x65 degree FOV for the depth sensor -->
         <horizontal_fov>1.5184351666666667</horizontal_fov>
         <vertical_fov>1.0122901111111111</vertical_fov>
@@ -27,5 +21,4 @@
         </image>
         <clip>
-          <!-- give the color sensor a maximum range of 50m so that the simulation renders nicely -->
           <near>0.01</near>
           <far>50.0</far>
@@ -68,5 +61,4 @@
   </link>
   <joint type="fixed" name="front_realsense_lens_joint">
-    <!-- Offset the camera 5cm forwards and 1cm up -->
     <origin xyz="0.05 0 0.01" rpy="0 0 0" />
     <parent link="front_mount" />
@@ -78,3 +70,53 @@
     <child link="front_realsense" />
   </joint>
+  <!-- Adding the Lidar -->
+  <link name="lidar_link">
+    <visual>
+      <origin xyz="0 0 0" rpy="0 0 0" />
+      <geometry>
+        <cylinder length="0.1" radius="0.05" />
+      </geometry>
+      <material name="grey" />
+    </visual>
+    <collision>
+      <origin xyz="0 0 0" rpy="0 0 0" />
+      <geometry>
+        <cylinder length="0.1" radius="0.05" />
+      </geometry>
+    </collision>
+  </link>
+  <joint name="lidar_joint" type="fixed">
+    <origin xyz="0.1 0 0.1" rpy="0 0 0" />
+    <parent link="front_mount" />
+    <child link="lidar_link" />
+  </joint>
+  <gazebo reference="lidar_link">
+    <sensor type="ray" name="lidar_sensor">
+      <update_rate>10</update_rate>
+      <ray>
+        <scan>
+          <horizontal>
+            <samples>360</samples>
+            <resolution>1</resolution>
+            <min_angle>-1.5708</min_angle>
+            <max_angle>1.5708</max_angle>
+          </horizontal>
+          <vertical>
+            <samples>1</samples>
+            <min_angle>0</min_angle>
+            <max_angle>0</max_angle>
+          </vertical>
+        </scan>
+        <range>
+          <min>0.1</min>
+          <max>10.0</max>
+          <resolution>0.01</resolution>
+        </range>
+      </ray>
+      <plugin name="gazebo_ros_laser" filename="libgazebo_ros_laser.so">
+        <topicName>/lidar/scan</topicName>
+        <frameName>lidar_link</frameName>
+      </plugin>
+    </sensor>
+  </gazebo>
 </robot>

Commit message: updated the lidar and commands used

File: catkin_ws/src/jackal_realsense/jackal_realsense.urdf.xacro (robot description, xacro)
@@ -1,4 +1,11 @@
 <?xml version="1.0"?>
 <robot xmlns:xacro="http://ros.org/wiki/xacro">
+  <!-- Material Definitions -->
+  <material name="white">
+    <color rgba="1 1 1 1"/>
+  </material>
+  <material name="grey">
+    <color rgba="0.5 0.5 0.5 1"/>
+  </material>
   <link name="front_realsense" />
   <link name="front_realsense_gazebo" />
@@ -38,14 +45,4 @@
         <pointCloudCutoff>0.105</pointCloudCutoff>
         <pointCloudCutoffMax>8.0</pointCloudCutoffMax>
-        <distortionK1>0.00000001</distortionK1>
-        <distortionK2>0.00000001</distortionK2>
-        <distortionK3>0.00000001</distortionK3>
-        <distortionT1>0.00000001</distortionT1>
-        <distortionT2>0.00000001</distortionT2>
-        <CxPrime>0</CxPrime>
-        <Cx>0</Cx>
-        <Cy>0</Cy>
-        <focalLength>0</focalLength>
-        <hackBaseline>0</hackBaseline>
       </plugin>
     </sensor>
